Commit message: trying to get AMCL working

File: kpbot_description/urdf/kpbot_base2.xacro (robot description, xacro)
@@ -30,5 +30,5 @@
     </link>
     <!-- Hokuyo Laser -->
-  <link name="laser">
+  <link name="base_scan">
     <collision>
       <origin xyz="0 0 0.0" rpy="0 0 1.57"/>
@@ -158,7 +158,7 @@
     <joint name="laser_joint" type="fixed">
         <axis xyz="0 1 0" />
-        <origin xyz="-0.03 0 0.145" rpy="0 0 0.0"/>
+        <origin xyz="-0.03 0 0.145" rpy="0 0 3.14"/>
         <parent link="base_link"/>
-        <child link="laser"/>
+        <child link="base_scan"/>
     </joint>
 </robot>
